Commit message: fixed rotations

File: rc_car/launch/ego_racecar.xacro (robot description, xacro)
@@ -73,5 +73,5 @@
     <child link="${car_name}/back_right_wheel"/>
     <origin xyz="0 ${-(wheel_length+width)/2} ${wheel_radius}" rpy="0 0 0" />
-    <axis xyz="0 -1 0"/>
+    <axis xyz="0 1 0"/>
   </joint>
   <link name="${car_name}/back_right_wheel">
@@ -123,10 +123,11 @@
     </gazebo>
   <!-- FRONT RIGHT HINGE -->
-  <joint name="base_to_front_right_hinge" type="continuous">
+  <joint name="base_to_front_right_hinge" type="revolute">
     <parent link="${car_name}/base_link"/>
     <child link="${car_name}/front_right_hinge"/>
     <origin xyz="${wheelbase} ${-(wheel_length+width)/2} ${wheel_radius}"/>
-    <axis xyz="0 0 -1"/>
-  </joint>
+    <axis xyz="0 0 1"/>
+    <limit effort="100" velocity="1" lower="-1" upper="1"/>
+    <dynamics damping="0.0" friction="0.0"/>  </joint>
   <link name="${car_name}/front_right_hinge">
  <visual>
@@ -150,10 +151,9 @@
     </gazebo>
   <!-- FRONT RIGHT WHEEL -->
-  <joint name="front_right_hinge_to_wheel" type="revolute">
+  <joint name="front_right_hinge_to_wheel" type="continuous">
     <parent link="${car_name}/front_right_hinge"/>
     <child link="${car_name}/front_right_wheel"/>
     <origin xyz="0 0 0"/>
-    <limit effort="100" velocity="1" lower="-1" upper="1"/>
-    <dynamics damping="0.0" friction="0.0"/>
+    <axis xyz="0 1 0"/>
   </joint>
   <link name="${car_name}/front_right_wheel">
@@ -178,10 +178,12 @@
     </gazebo>
   <!-- FRONT LEFT HINGE -->
-  <joint name="base_to_front_left_hinge" type="continuous">
+  <joint name="base_to_front_left_hinge" type="revolute">
     <parent link="${car_name}/base_link"/>
     <child link="${car_name}/front_left_hinge"/>
     <origin xyz="${wheelbase} ${(wheel_length+width)/2} ${wheel_radius}"/>
     <axis xyz="0 0 1"/>
-  </joint>
+    <limit effort="100" velocity="1" lower="-1" upper="1"/>
+    <dynamics damping="0.0" friction="0.0"/>
+    </joint>
   <link name="${car_name}/front_left_hinge" >
    <visual>
@@ -205,10 +207,9 @@
     </gazebo>
   <!-- FRONT LEFT WHEEL -->
-  <joint name="front_left_hinge_to_wheel" type="revolute">
+  <joint name="front_left_hinge_to_wheel" type="continuous">
     <parent link="${car_name}/front_left_hinge"/>
     <child link="${car_name}/front_left_wheel"/>
     <origin xyz="0 0 0"/>
-    <limit effort="100" velocity="1" lower="-1" upper="1"/>
-    <dynamics damping="0.0" friction="0.0"/>
+    <axis xyz="0 1 0"/>
   </joint>
   <link name="${car_name}/front_left_wheel">

Commit message: added teleop, fixed hinge sizes

File: rc_car/launch/ego_racecar.xacro (robot description, xacro)
@@ -133,11 +133,11 @@
  <visual>
       <geometry>
-        <cylinder radius="${wheel_radius}" length="${wheel_length}"/>
-      </geometry>
-      <origin rpy="-${pi/2} 0 0"/>
-    </visual>
-    <collision>
-      <geometry>
-        <cylinder radius="${wheel_radius}" length="${wheel_length}"/>
+        <cylinder radius="${wheel_radius/4}" length="${wheel_length/4}"/>
+      </geometry>
+      <origin rpy="-${pi/2} 0 0"/>
+    </visual>
+    <collision>
+      <geometry>
+        <cylinder radius="${wheel_radius/4}" length="${wheel_length/4}"/>
       </geometry>
       <origin rpy="-${pi/2} 0 0"/>
@@ -189,11 +189,11 @@
    <visual>
       <geometry>
-        <cylinder radius="${wheel_radius}" length="${wheel_length}"/>
-      </geometry>
-      <origin rpy="${pi/2} 0 0"/>
-    </visual>
-    <collision>
-      <geometry>
-        <cylinder radius="${wheel_radius}" length="${wheel_length}"/>
+        <cylinder radius="${wheel_radius/4}" length="${wheel_length/4}"/>
+      </geometry>
+      <origin rpy="${pi/2} 0 0"/>
+    </visual>
+    <collision>
+      <geometry>
+        <cylinder radius="${wheel_radius/4}" length="${wheel_length/4}"/>
       </geometry>
       <origin rpy="${pi/2} 0 0"/>
@@ -218,5 +218,5 @@
         <cylinder radius="${wheel_radius}" length="${wheel_length}"/>
       </geometry>
-      <origin rpy="${pi/2} 0 0"/>
+      <origin xyz="0 0.005 0" rpy="${pi/2} 0 0"/>
     </visual>
     <collision>
