Commit message: Tried various models with ackermann steering. No bite

File: rc_car/description/gazebo_control.xacro (robot description, xacro)
@@ -1,21 +1,22 @@
 <?xml version="1.0"?>
 <robot xmlns:xacro="http://www.ros.org/wiki/xacro">
-  <gazebo>
-    <plugin name="diff_drive" filename="libgazebo_ros_diff_drive.so">
-      <!-- Wheel Information -->
-      <left_joint>left_wheel_joint</left_joint>
-      <right_joint>right_wheel_joint</right_joint>
-      <wheel_separation>0.35</wheel_separation>
-      <wheel_diameter>0.1</wheel_diameter>
-      <!-- Limits -->
-      <max_wheel_torque>200</max_wheel_torque>
-      <max_wheel_acceleration>10.0</max_wheel_acceleration>
-      <!-- Output -->
-      <odometry_frame>odom</odometry_frame>
-      <robot_base_frame>base_link</robot_base_frame>
-      <publish_odom>true</publish_odom>
-      <publish_odom_tf>true</publish_odom_tf>
-      <publish_wheel_tf>true</publish_wheel_tf>
-    </plugin>
-  </gazebo>
+    <gazebo>
+        <plugin name="diff_drive" filename="libgazebo_ros_diff_drive.so">
+          <update_rate>100.0</update_rate>
+            <!-- Wheel Information -->
+            <left_joint>left_wheel_joint</left_joint>
+            <right_joint>right_wheel_joint</right_joint>
+            <wheel_separation>0.35</wheel_separation>
+            <wheel_diameter>0.1</wheel_diameter>
+            <!-- Limits -->
+            <max_wheel_torque>200</max_wheel_torque>
+            <max_wheel_acceleration>10.0</max_wheel_acceleration>
+            <!-- Output -->
+            <odometry_frame>odom</odometry_frame>
+            <robot_base_frame>base_link</robot_base_frame>
+            <publish_odom>true</publish_odom>
+            <publish_odom_tf>true</publish_odom_tf>
+            <publish_wheel_tf>true</publish_wheel_tf>
+        </plugin>
+    </gazebo>
 </robot>

File: rc_car/description/robot.urdf.xacro (robot description, xacro)
@@ -1,4 +1,4 @@
 <?xml version="1.0"?>
-<robot xmlns:xacro="http://www.ros.org/wiki/xacro" name="robot">
+<robot xmlns:xacro="http://www.ros.org/wiki/xacro"  name="robot">
     <xacro:include filename="robot_core.xacro" />
     <xacro:include filename="gazebo_control.xacro" />

File: rc_car/description/robot_core.xacro (robot description, xacro)
@@ -1,4 +1,4 @@
 <?xml version="1.0"?>
-<robot xmlns:xacro="http://www.ros.org/wiki/xacro">
+<robot xmlns:xacro="http://www.ros.org/wiki/xacro" >
     <xacro:include filename="inertial_macros.xacro"/>
     <material name="white">

File: rc_car/launch/em.urdf.xacro (robot description, xacro)
@@ -1,336 +1,17 @@
 <?xml version="1.0"?>
-<robot name="ackermann_1"
-  xmlns:xacro="http://www.ros.org/wiki/xacro">
-  <xacro:include filename="gazebo_control.xacro"/>
-  <!-- Base link -->
-  <link name="base_link">
-    <visual>
-      <geometry>
-        <box size="0.01 0.01 0.01"/>
-      </geometry>
-    </visual>
-  </link>
-  <!-- Chassis START-->
-  <joint name="base_joint" type="fixed">
-    <parent link="base_link"/>
-    <child link="chassis"/>
-  </joint>
-  <link name="chassis">
-    <collision>
-      <origin xyz="0 0 0.3" rpy="0 0 0"/>
-      <geometry>
-        <box size="1 0.2 0.1"/>
-      </geometry>
-    </collision>
-    <visual>
-      <origin xyz="0 0 0.3" rpy="0 0 0"/>
-      <geometry>
-        <box size="1 0.2 0.1"/>
-      </geometry>
-      <material name="orange"/>
-    </visual>
-    <inertial>
-      <mass value="1"/>
-      <origin xyz="0 0 0.3" rpy="0 0 0"/>
-      <inertia ixx="0.4" ixy="0.1" ixz="0.1" iyy="0.4" iyz="0.1" izz="0.2"/>
-    </inertial>
-  </link>
-  <joint name="steering_wheel_joint" type="revolute">
-    <parent link="some_parent_link"/>
-    <child link="steering_wheel_link"/>
-    <origin xyz="0 0 0" rpy="0 0 0"/>
-    <axis xyz="0 0 1"/>
-    <limit effort="100" velocity="1" lower="-1" upper="1"/>
-    <dynamics damping="0.0" friction="0.0"/>
-  </joint>
-  <gazebo reference="chassis">
-    <!--Stiffness -->
-    <kp>1000000.0</kp>
-    <!--Dampening-->
-    <kd>0.1</kd>
-    <dampingFactor>0</dampingFactor>
-    <material>Gazebo/White</material>
-    <selfCollide>true</selfCollide>
-    <turnGravityOff>false</turnGravityOff>
-    <mu1 value="0.1"/>
-    <mu2 value="0.1"/>
-    <fdir1 value="0 0 0"/>
-  </gazebo>
-  <!-- Chassis END -->
-  <!-- Right Wheel - Start -->
-  <link name="right_wheel">
-    <collision>
-      <origin xyz="0 0 0" rpy="0 1.5708 1.5708" />
-      <geometry>
-        <cylinder length="0.05" radius="0.1"/>
-      </geometry>
-    </collision>
-    <visual>
-      <origin xyz="0 0 0" rpy="0 1.5708 1.5708" />
-      <geometry>
-        <cylinder length="0.05" radius="0.1"/>
-      </geometry>
-      <material name="black"/>
-    </visual>
-    <inertial>
-      <origin xyz="0 0 0" rpy="0 1.5708 1.5708" />
-      <mass value="0.2"/>
-      <cylinder_inertia m="0.2" r="0.3" h="0.1"/>
-      <inertia ixx="0.4" ixy="0.1" ixz="0.1" iyy="0.4" iyz="0.1" izz="0.2"/>
-    </inertial>
-  </link>
-  <gazebo reference="right_wheel">
-    <mu1 value="2.0"/>
-    <mu2 value="2.0"/>
-    <kp value="10000000.0" />
-    <kd value="1.0" />
-    <fdir1 value="0 1 0"/>
-    <material>Gazebo/Blue</material>
-  </gazebo>
-  <link name="right_wheel_assembly">
-    <collision>
-      <origin xyz="0 0 0" rpy="0 1.5708 1.5708" />
-      <geometry>
-        <cylinder length="0.001" radius="0.04"/>
-      </geometry>
-    </collision>
-    <visual>
-      <origin xyz="0 0 0" rpy="0 1.5708 1.5708" />
-      <geometry>
-        <cylinder length="0.001" radius="0.04"/>
-      </geometry>
-      <material name="white"/>
-    </visual>
-    <inertial>
-      <origin xyz="0 0 0" rpy="0 1.5708 1.5708" />
-      <mass value="0.2"/>
-      <cylinder_inertia m="0.2" r="0.3" h="0.1"/>
-      <inertia ixx="0.4" ixy="0.1" ixz="0.1" iyy="0.4" iyz="0.1" izz="0.2"/>
-    </inertial>
-  </link>
-  <gazebo reference="right_wheel_assembly">
-    <mu1 value="2.0"/>
-    <mu2 value="2.0"/>
-    <kp value="10000000.0" />
-    <kd value="1.0" />
-    <fdir1 value="0 1 0"/>
-    <material>Gazebo/White</material>
-  </gazebo>
-  <joint name="right_wheel_hinge" type="revolute">
-    <parent link="chassis"/>
-    <child link="right_wheel_assembly"/>
-    <origin xyz="0.4 0.125 0.3" rpy="0 0 0" />
-    <axis xyz="0 0 1" rpy="0 0 0" />
-    <limit effort="100" velocity="1" lower="-1" upper="1"/>
-    <dynamics damping="0.0" friction="0.0"/>
-  </joint>
-  <joint name="right_wheel_rotate" type="continuous">
-    <parent link="right_wheel_assembly"/>
-    <child link="right_wheel"/>
-    <origin xyz="0.0 0.025 0.0" rpy="0 0 0" />
-    <axis xyz="0 1 0" rpy="0 0 0" />
-    <limit effort="100" velocity="50"/>
-    <dynamics damping="0.0" friction="0.0"/>
-  </joint>
-  <transmission name="trans_right_wheel_hing">
-    <type>transmission_interface/SimpleTransmission</type>
-    <joint name="right_wheel_hinge">
-      <hardwareInterface>EffortJointInterface</hardwareInterface>
-    </joint>
-    <actuator name="motor1">
-      <hardwareInterface>EffortJointInterface</hardwareInterface>
-      <mechanicalReduction>1</mechanicalReduction>
-    </actuator>
-  </transmission>
-  <transmission name="trans_right_wheel_rotate">
-    <type>transmission_interface/SimpleTransmission</type>
-    <joint name="right_wheel_rotate">
-      <hardwareInterface>EffortJointInterface</hardwareInterface>
-    </joint>
-    <actuator name="motor_right_wheel_rotate">
-      <hardwareInterface>EffortJointInterface</hardwareInterface>
-      <mechanicalReduction>1</mechanicalReduction>
-    </actuator>
-  </transmission>
-  <!-- Right Wheel - End -->
-  <!-- Left Wheel - Start  -->
-  <link name="left_wheel">
-    <collision>
-      <origin xyz="0 0 0" rpy="0 1.5708 1.5708" />
-      <geometry>
-        <cylinder length="0.05" radius="0.1"/>
-      </geometry>
-    </collision>
-    <visual>
-      <origin xyz="0 0 0" rpy="0 1.5708 1.5708" />
-      <geometry>
-        <cylinder length="0.05" radius="0.1"/>
-      </geometry>
-      <material name="black"/>
-    </visual>
-    <inertial>
-      <origin xyz="0 0 0" rpy="0 1.5708 1.5708" />
-      <mass value="0.2"/>
-      <cylinder_inertia m="0.2" r="0.3" h="0.1"/>
-      <inertia ixx="0.4" ixy="0.1" ixz="0.1" iyy="0.4" iyz="0.1" izz="0.2"/>
-    </inertial>
-  </link>
-  <gazebo reference="left_wheel">
-    <mu1 value="2.0"/>
-    <mu2 value="2.0"/>
-    <kp value="10000000.0" />
-    <kd value="1.0" />
-    <fdir1 value="0 1 0"/>
-    <material>Gazebo/Blue</material>
-  </gazebo>
-  <link name="left_wheel_assembly">
-    <collision>
-      <origin xyz="0 0 0" rpy="0 1.5708 1.5708" />
-      <geometry>
-        <cylinder length="0.001" radius="0.04"/>
-      </geometry>
-    </collision>
-    <visual>
-      <origin xyz="0 0 0" rpy="0 1.5708 1.5708" />
-      <geometry>
-        <cylinder length="0.001" radius="0.04"/>
-      </geometry>
-      <material name="white"/>
-    </visual>
-    <inertial>
-      <origin xyz="0 0 0" rpy="0 1.5708 1.5708" />
-      <mass value="0.2"/>
-      <cylinder_inertia m="0.2" r="0.3" h="0.1"/>
-      <inertia ixx="0.4" ixy="0.1" ixz="0.1" iyy="0.4" iyz="0.1" izz="0.2"/>
-    </inertial>
-  </link>
-  <gazebo reference="left_wheel_assembly">
-    <mu1 value="2.0"/>
-    <mu2 value="2.0"/>
-    <kp value="10000000.0" />
-    <kd value="1.0" />
-    <fdir1 value="0 1 0"/>
-    <material>Gazebo/White</material>
-  </gazebo>
-  <joint name="left_wheel_hinge" type="revolute">
-    <parent link="chassis"/>
-    <child link="left_wheel_assembly"/>
-    <origin xyz="0.4 -0.125 0.3" rpy="0 0 0" />
-    <axis xyz="0 0 1" rpy="0 0 0" />
-    <limit effort="100" velocity="1" lower="-1" upper="1"/>
-    <dynamics damping="0.0" friction="0.0"/>
-  </joint>
-  <joint name="left_wheel_rotate" type="continuous">
-    <parent link="left_wheel_assembly"/>
-    <child link="left_wheel"/>
-    <origin xyz="0.0 -0.025 0.0" rpy="0 0 0" />
-    <axis xyz="0 1 0" rpy="0 0 0" />
-    <limit effort="0" velocity="0"/>
-    <dynamics damping="0.0" friction="0.0"/>
-  </joint>
-  <transmission name="tran2">
-    <type>transmission_interface/SimpleTransmission</type>
-    <joint name="left_wheel_hinge">
-      <hardwareInterface>EffortJointInterface</hardwareInterface>
-    </joint>
-    <actuator name="motor2">
-      <hardwareInterface>EffortJointInterface</hardwareInterface>
-      <mechanicalReduction>1</mechanicalReduction>
-    </actuator>
-  </transmission>
-  <transmission name="trans_left_wheel_rotate">
-    <type>transmission_interface/SimpleTransmission</type>
-    <joint name="left_wheel_rotate">
-      <hardwareInterface>EffortJointInterface</hardwareInterface>
-    </joint>
-    <actuator name="motor_left_wheel_rotate">
-      <hardwareInterface>EffortJointInterface</hardwareInterface>
-      <mechanicalReduction>1</mechanicalReduction>
-    </actuator>
-  </transmission>
-  <!-- Left Wheel - End -->
-  <!-- Right Rear Wheel Start -->
-  <link name="right_wheel_rear">
-    <collision>
-      <origin xyz="0 0 0" rpy="0 1.5708 1.5708" />
-      <geometry>
-        <cylinder length="0.05" radius="0.1"/>
-      </geometry>
-    </collision>
-    <visual>
-      <origin xyz="0 0 0" rpy="0 1.5708 1.5708" />
-      <geometry>
-        <cylinder length="0.05" radius="0.1"/>
-      </geometry>
-      <material name="black"/>
-    </visual>
-    <inertial>
-      <origin xyz="0 0 0" rpy="0 1.5708 1.5708" />
-      <mass value="0.2"/>
-      <cylinder_inertia m="0.2" r="0.3" h="0.1"/>
-      <inertia ixx="0.4" ixy="0.1" ixz="0.1" iyy="0.4" iyz="0.1" izz="0.2"/>
-    </inertial>
-  </link>
-  <joint name="right_wheel_rear_rotate" type="continuous">
-    <parent link="chassis"/>
-    <child link="right_wheel_rear"/>
-    <origin xyz="-0.4 0.15 0.3" rpy="0 0 0" />
-    <axis xyz="0 1 0" rpy="0 0 0" />
-    <limit effort="0" velocity="0"/>
-    <dynamics damping="0.0" friction="0.0"/>
-  </joint>
-  <gazebo reference="right_wheel_rear">
-    <mu1 value="2.0"/>
-    <mu2 value="2.0"/>
-    <kp value="10000000.0" />
-    <kd value="1.0" />
-    <fdir1 value="0 1 0"/>
-    <material>Gazebo/Blue</material>
-  </gazebo>
-  <!-- Right Rear Wheel End -->
-  <!-- Right Rear Wheel Start -->
-  <link name="left_wheel_rear">
-    <collision>
-      <origin xyz="0 0 0" rpy="0 1.5708 1.5708" />
-      <geometry>
-        <cylinder length="0.05" radius="0.1"/>
-      </geometry>
-    </collision>
-    <visual>
-      <origin xyz="0 0 0" rpy="0 1.5708 1.5708" />
-      <geometry>
-        <cylinder length="0.05" radius="0.1"/>
-      </geometry>
-      <material name="black"/>
-    </visual>
-    <inertial>
-      <origin xyz="0 0 0" rpy="0 1.5708 1.5708" />
-      <mass value="0.2"/>
-      <cylinder_inertia m="0.2" r="0.3" h="0.1"/>
-      <inertia ixx="0.4" ixy="0.1" ixz="0.1" iyy="0.4" iyz="0.1" izz="0.2"/>
-    </inertial>
-  </link>
-  <joint name="left_wheel_rear_rotate" type="continuous">
-    <parent link="chassis"/>
-    <child link="left_wheel_rear"/>
-    <origin xyz="-0.4 -0.15 0.3" rpy="0 0 0" />
-    <axis xyz="0 1 0" rpy="0 0 0" />
-    <limit effort="0" velocity="0"/>
-    <dynamics damping="0.0" friction="0.0"/>
-  </joint>
-  <gazebo reference="left_wheel_rear">
-    <mu1 value="2.0"/>
-    <mu2 value="2.0"/>
-    <kp value="10000000.0" />
-    <kd value="1.0" />
-    <fdir1 value="0 1 0"/>
-    <material>Gazebo/Blue</material>
-  </gazebo>
-  <!-- Left Rear Wheel End -->
-  <!-- <gazebo>
-    <plugin name="gazebo_ros_control" filename="libgazebo_ros_control.so">
-      <robotNamespace>/ack</robotNamespace>
-      <legacyModeNS>true</legacyModeNS>
-    </plugin>
-  </gazebo> -->
+<!-- 4 Wheel Robot with front steering and rear drive -->
+<robot xmlns:xacro="http://www.ros.org/wiki/xacro" name="carlikebot_robot">
+  <xacro:arg name="prefix" default="" />
+  <xacro:include filename="gazebo_control.xacro" />
+  <xacro:include
+    filename="$(find rc_car)/launch/carlikebot_description.urdf.xacro" />
+  <!-- Import Rviz colors -->
+  <xacro:include
+    filename="$(find rc_car)/launch/carlikebot.materials.xacro" />
+  <!-- Import carlikebot ros2_control description -->
+  <xacro:include
+    filename="$(find rc_car)/launch/carlikebot.ros2_control.xacro" />
+  <xacro:carlikebot prefix="$(arg prefix)" />
+  <xacro:carlikebot_ros2_control
+    name="CarlikeBot" prefix="$(arg prefix)" />
 </robot>

File: rc_car/launch/gazebo_control.xacro (robot description, xacro)
@@ -1,36 +1,44 @@
 <?xml version="1.0"?>
 <robot xmlns:xacro="http://www.ros.org/wiki/xacro">
-  <gazebo>
-    <plugin name="gazebo_ros_ackermann_drive" filename="libgazebo_ros_ackermann_drive.so">
-      <!-- wheels -->
-      <front_left_joint>base_to_front_left_hinge</front_left_joint>
-      <front_right_joint>base_to_front_right_hinge</front_right_joint>
-      <rear_left_joint>base_to_back_left_wheel</rear_left_joint>
-      <rear_right_joint>base_to_back_right_wheel</rear_right_joint>
-      <left_steering_joint>front_left_hinge_to_wheel</left_steering_joint>
-      <right_steering_joint>front_right_hinge_to_wheel</right_steering_joint>
-      <!-- <steering_wheel_joint>steering_joint</steering_wheel_joint> -->
-      <!-- Max absolute steer angle for tyre in radians-->
-      <!-- Any cmd_vel angular z greater than this would be capped -->
-      <max_steer>0.6458</max_steer>
-      <!-- Max absolute steering angle of steering wheel -->
-      <max_steering_angle>7.85</max_steering_angle>
-      <!-- Max absolute linear speed in m/s -->
-      <max_speed>20</max_speed>
-      <!-- PID tuning -->
-      <left_steering_pid_gain>1500 0 1</left_steering_pid_gain>
-      <left_steering_i_range>0 0</left_steering_i_range>
-      <right_steering_pid_gain>1500 0 1</right_steering_pid_gain>
-      <right_steering_i_range>0 0</right_steering_i_range>
-      <linear_velocity_pid_gain>1000 0 1</linear_velocity_pid_gain>
-      <linear_velocity_i_range>0 0</linear_velocity_i_range>
-      <!-- output -->
-      <publish_odom>true</publish_odom>
-      <publish_odom_tf>true</publish_odom_tf>
-      <publish_wheel_tf>true</publish_wheel_tf>
-      <publish_distance>true</publish_distance>
-      <odometry_frame>odom_demo</odometry_frame>
-      <robot_base_frame>chassis</robot_base_frame>
-    </plugin>
-  </gazebo>
+  <xacro:macro name="carlikebot" params="prefix">
+    <gazebo>
+      <plugin name="gazebo_ros_ackermann_drive" filename="libgazebo_ros_ackermann_drive.so">
+        <ros>
+          <parameter name="cmd_vel_topic" value="cmd_demo" />
+          <parameter name="odom_topic" value="odom_demo" />
+          <parameter name="distance_topic" value="distance_demo" />
+        </ros>
+        <update_rate>100.0</update_rate>
+        <!-- wheels -->
+        <front_left_joint>virtual_rear_wheel_joint</front_left_joint>
+        <front_right_joint>virtual_rear_wheel_joint</front_right_joint>
+        <rear_left_joint>virtual_rear_wheel_joint</rear_left_joint>
+        <rear_right_joint>virtual_rear_wheel_joint</rear_right_joint>
+        <left_steering_joint>virtual_front_wheel_joint</left_steering_joint>
+        <right_steering_joint>virtual_front_wheel_joint</right_steering_joint>
+        <!-- <steering_wheel_joint>steering_joint</steering_wheel_joint> -->
+        <!-- Max absolute steer angle for tyre in radians-->
+        <!-- Any cmd_vel angular z greater than this would be capped -->
+        <max_steer>0.6458</max_steer>
+        <!-- Max absolute steering angle of steering wheel -->
+        <max_steering_angle>7.85</max_steering_angle>
+        <!-- Max absolute linear speed in m/s -->
+        <max_speed>20</max_speed>
+        <!-- PID tuning -->
+        <left_steering_pid_gain>1500 0 1</left_steering_pid_gain>
+        <left_steering_i_range>0 0</left_steering_i_range>
+        <right_steering_pid_gain>1500 0 1</right_steering_pid_gain>
+        <right_steering_i_range>0 0</right_steering_i_range>
+        <linear_velocity_pid_gain>1000 0 1</linear_velocity_pid_gain>
+        <linear_velocity_i_range>0 0</linear_velocity_i_range>
+        <!-- output -->
+        <publish_odom>true</publish_odom>
+        <publish_odom_tf>true</publish_odom_tf>
+        <publish_wheel_tf>true</publish_wheel_tf>
+        <publish_distance>true</publish_distance>
+        <odometry_frame>odom_demo</odometry_frame>
+        <robot_base_frame>chassis</robot_base_frame>
+      </plugin>
+    </gazebo>
+  </xacro:macro>
 </robot>
